File: Hardware/CH340/USB-RS485_CH340.kicad_sch (KiCad schematic)
At the start: 39 parts, among them J2 7-pin con, J3 3.3 LVL 5, J6 USB_C_Receptacle_USB2.0_16P, Q1 BC857, U1 CH340G, U2 SN75176AD, U3 AMS1117-3.3, U4 DC-DC, U5 EL817, U6 EL817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

Commit message: schematics cosmetic change
Other:
- note added: "ISOLATED PART"
- note added: "NON-ISOLATED PART"
- moved on the sheet: C1, C2, C3, C4, C5, C6, C7, C8, C9, D1, D2, D3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
