File: Hardware/FT230/USB-RS485_FT230.kicad_pcb (KiCad board)
At the start: 2 copper layers, 59 x 22.5 mm, 35 parts, among them J1 USB_C_Receptacle_USB2.0_16P, J2 7-pin con, J4 Conn_02x04_Odd_Even, U1 FT230XQ, U2 ADuM121N, U3 DC-DC, U4 ISO3082DW, U5 AP7345D-1833RH4-7

Commit message: layout update
Parts:
- removed J4: Conn_02x04_Odd_Even, Connector_PinHeader_2.54mm:PinHeader_2x04_P2.54mm_Vertical
- added C16: 100nF, Capacitor_SMD:C_0805_2012Metric, F.Cu at (164.5, 87.9)
- added J3: 7-pin con, Connector_PinHeader_2.54mm:PinHeader_1x07_P2.54mm_Vertical, F.Cu at (172.7, 86.0)
- added R9: 10k, Resistor_SMD:R_0805_2012Metric, F.Cu at (135.7, 85.7)
- added REF**: OSHW-Logo2_7.3x6mm_SilkScreen, Symbol:OSHW-Logo2_7.3x6mm_SilkScreen, B.Cu at (168.1, 93.6)
- added U6: AP7345D-1833RH4-7, AP7345D-1833:AP7345D1833RH47, F.Cu at (164.5, 85.6)
- C1: value 4.7uF -> 47pF
- C10: value 100nF -> 270pF/2kV; footprint Capacitor_SMD:C_0805_2012Metric -> Capacitor_SMD:C_1206_3216Metric; moved to B.Cu
- C11: value 10uF -> 100nF
- C13: value 100nF -> 10uF
- C2: value 47pF -> 4.7uF
- C3: value 100nF -> 47pF
- C4: value 47pF -> 100nF
- C6: value 4.7uF -> 100nF
- C7: value 100nF -> 4.7uF
- C9: value 270pF/2kV -> 100nF; footprint Capacitor_SMD:C_1206_3216Metric -> Capacitor_SMD:C_0805_2012Metric
- J2: value 7-pin con -> Conn_02x04_Odd_Even; footprint Connector_PinHeader_2.54mm:PinHeader_1x07_P2.54mm_Vertical -> Connector_PinHeader_2.54mm:PinHeader_2x04_P2.54mm_Vertical
- U2: value ADuM121N -> TS5A3159DCK; footprint Package_SO:SOIC-8_3.9x4.9mm_P1.27mm -> Package_TO_SOT_SMD:SOT-363_SC-70-6
- U3: value DC-DC -> ADuM121N; footprint Converter_DCDC:Converter_DCDC_TRACO_TEA1-xxxx_THT -> Package_SO:SOIC-8_3.9x4.9mm_P1.27mm
- U4: value ISO3082DW -> DC-DC; footprint Package_SO:SOIC-16W_7.5x10.3mm_P1.27mm -> Converter_DCDC:Converter_DCDC_TRACO_TEA1-xxxx_THT
- U5: value AP7345D-1833RH4-7 -> ISO3082DWR; footprint AP7345D-1833:AP7345D1833RH47 -> Package_SO:SOIC-16W_7.5x10.3mm_P1.27mm; moved to B.Cu
- moved C10 94.9 mm to (154.3, 100.3)
- moved J2 91.9 mm to (160.6, 84.1), turned to -90 degrees
- moved C13 89.2 mm to (163.7, 102.0), turned to 90 degrees
- moved C11 87.8 mm to (164.6, 90.5)
- moved C12 86.8 mm to (161.5, 98.1), turned to 90 degrees
- moved C14 86.0 mm to (161.5, 102.1), turned to 90 degrees
- moved C6 83.3 mm to (144.9, 93.1), turned to -90 degrees
- moved C15 82.7 mm to (164.6, 83.4), turned to 180 degrees
- moved R7 73.7 mm to (166.1, 93.6), turned to 90 degrees
- moved R8 71.8 mm to (163.7, 98.0), turned to -90 degrees
- moved D1 71.0 mm to (144.5, 101.8)
- moved C5 70.9 mm to (138.9, 88.2), turned to 90 degrees
- moved C3 70.1 mm to (135.7, 96.7), turned to 180 degrees
- moved C2 69.8 mm to (135.6, 87.9), turned to 0 degrees
- moved C4 69.8 mm to (135.7, 98.9), turned to 0 degrees
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Connections:
- C1 pad 1: GND1 -> Net-(U1-USBDP)
- C1 pad 2: +5V_USB -> GND1
- C10 pad 1: +V_OUT -> GND1
- C11 pad 1: Net-(U3--Vout) -> +V_OUT
- C11 pad 2: +5V_ISO -> GND2
- C13 pad 1: Net-(U3--Vout) -> GND2
- C14 pad 2: +1.8V_ISO -> +5V_ISO
- C15 pad 2: +3.3V_ISO -> +1.8V_ISO
- C2 pad 1: Net-(U1-USBDP) -> GND1
- C2 pad 2: GND1 -> +5V_USB
- C3 pad 1: +5V_USB -> Net-(U1-USBDM)
- C4 pad 1: Net-(U1-USBDM) -> +5V_USB
- C6 pad 1: GND1 -> VCCIO
- C6 pad 2: +5V_USB -> GND1
- C7 pad 2: Net-(U4-Vcc1) -> +5V_USB
- C9 pad 2: Net-(U3--Vout) -> VCCIO
- D3 pad 1: Net-(D3-A1) -> /RS485_P
- D3 pad 2: Net-(D3-A2) -> /RS485_N
- J2 pad 1: GND2 -> +1.8V_ISO
- J2 pad 2: Net-(D3-A1) -> +V_OUT
- J2 pad 3: Net-(D3-A2) -> +3.3V_ISO
- J2 pad 4: Net-(J2-Pin_4) -> +V_OUT
- J2 pad 5: Net-(J2-Pin_5) -> +5V_ISO
- J2 pad 7: GND2 -> VCCIO
- R7 pad 1: Net-(D3-A2) -> /RS485_N
- R7 pad 2: Net-(D3-A1) -> /RS485_P
- U2 pad 1: VCCIO -> Net-(U5-R)
- U2 pad 2: Net-(U1-RXD) -> GND1
- U2 pad 3: Net-(U1-TXD) -> Net-(U3-VOA)
- U2 pad 4: GND1 -> Net-(U1-RXD)
- U2 pad 5: GND2 -> VCCIO
- U2 pad 6: Net-(J2-Pin_4) -> RS_ACT
- U3 pad 1: GND1 -> VCCIO
- U3 pad 2: +5V_USB -> Net-(U3-VOA)
- U3 pad 3: Net-(U3--Vout) -> Net-(U1-TXD)
- U3 pad 4: +5V_ISO -> GND1
- U4 pad 1: Net-(U4-Vcc1) -> GND1
- U4 pad 2: GND1 -> +5V_USB
- U4 pad 3: Net-(U1-RXD) -> GND2
- U4 pad 4: Net-(U1-CBUS3) -> +5V_ISO
- U5 pad 1: GND2 -> VCCIO
- U5 pad 2: +1.8V_ISO -> GND1
- U5 pad 3: +3.3V_ISO -> Net-(U5-R)
- U5 pad 4: GND2 -> Net-(U1-CBUS3)
- U5 pad 5: +5V_ISO -> Net-(U1-CBUS2)
- U5 pad 6: +5V_ISO -> Net-(U1-TXD)
- U5 pad 7: +5V_ISO -> GND1
- U5 pad 8: +5V_ISO -> GND1
Routing:
- net VCCIO: track 24.1 -> 71.6 mm, vias 2 -> 5
- net +5V_ISO: track 0.00 -> 45.7 mm, vias 0 -> 1
- net +V_OUT: track 0.00 -> 42.3 mm, vias 0 -> 2
- net +5V_USB: track 31.3 -> 59.1 mm
- net RS_ACT: track 0.00 -> 23.5 mm
- net GND2: track 0.00 -> 22.3 mm, vias 0 -> 10
- net /RS485_N: track 0.00 -> 18.0 mm, vias 0 -> 1
- net /RS485_P: track 0.00 -> 17.9 mm, vias 0 -> 1
- net Net-(J3-Pin_4): track 0.00 -> 17.5 mm
- net Net-(J3-Pin_5): track 0.00 -> 16.5 mm
- net Net-(U5-R): track 0.00 -> 14.8 mm, vias 0 -> 1
- net Net-(U1-CBUS2): track 0.00 -> 14.2 mm, vias 0 -> 3
- net Net-(U3-VOA): track 0.00 -> 14.1 mm
- net Net-(U1-RXD): track 11.6 -> 2.38 mm
- net +3.3V_ISO: track 0.00 -> 8.76 mm
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Other:
- board size 59 x 22.5 mm -> 50 x 23 mm
- board text added: "1.8V"
- board text added: "3.3V"
- board text added: "5V"
- board text added: "A"
- board text added: "B"
- board text added: "GND"
- board text added: "RS485"
- board text added: "Rx"
- board text added: "Tx"
- board text added: "Vcc"
- board text added: "github.com/even-notodd/ISO-RS485"
- board text removed: "USB-UART/RS485 (GALVANIC ISOLATION)"
