File: Hardware/FT230/USB-RS485_FT230.kicad_pcb (KiCad board)
At the start: 2 copper layers, 50 x 23 mm, 39 parts, among them J1 USB_C_Receptacle_USB2.0_16P, J2 Conn_02x04_Odd_Even, J3 7-pin con, U1 FT230XQ, U2 TS5A3159DCK, U3 ADuM121N, U4 DC-DC, U5 ISO3082DWR, U6 AP7345D-1833RH4-7

Commit message: CBUS-configs
Parts:
- removed REF**: OSHW-Logo2_7.3x6mm_SilkScreen, Symbol:OSHW-Logo2_7.3x6mm_SilkScreen
