File: Hardware/FT230/USB-RS485_FT230.kicad_sch (KiCad schematic)
At the start: 37 parts, among them J1 USB_C_Receptacle_USB2.0_16P, J2 7-pin con, J4 Conn_02x04_Odd_Even, U1 FT230XQ, U2 ADuM121N, U3 DC-DC, U4 ISO3082DWR, U5 AP7345D-1833RH4-7, U6 TS5A3159DCK

Commit message: layout update
Parts:
- added R9: 10k, Resistor_SMD:R_0805_2012Metric, symbol Device:R
- U6: renamed from U5; footprint AP7345D1833RH47 -> AP7345D-1833:AP7345D1833RH47
- renumbered C2 to C1, C9 to C10, C10 to C11, C11 to C13, C13 to C14, C14 to C15, C15 to C16, C1 to C2, C4 to C3, C3 to C4, C16 to C5, C5 to C6, C6 to C7, C7 to C9, J4 to J2, J2 to J3, U6 to U2, U2 to U3, U3 to U4, U4 to U5
Connections:
- net GND1: now also R9.2
- net GND2: now also C10.2, C13.1, C14.1, U4.3 (-Vout)
- net RS_ACT: now also R9.1
- net RS485_P: now reaches D3.1 (A1), J3.2 (Pin_2), R7.2, U5.12 (A)
- net RS485_N: now reaches D3.2 (A2), J3.3 (Pin_3), R7.1, U5.13 (B)
- net at U3.6 (VOB): now also J3.5 (Pin_5); no longer J3.4 (Pin_4)
- net at U3.7 (VIA): now also J3.4 (Pin_4); no longer J3.5 (Pin_5)

Commit message: CBUS-configs
Parts:
- U2: MPN (none) -> TS5A3159DCK; Manufacturer (none) -> TI
Changed lines of the file:
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@@
+			)
+		)
+		(property "Manufacturer" "TI"
+			(at 132.08 38.1 0)
+			(effects
+				(font
+					(size 1.27 1.27)
+				)
+				(hide yes)
+			)
+		)
+		(property "MPN" "TS5A3159DCK"
+			(at 132.08 38.1 0)
+			(effects
+				(font
+					(size 1.27 1.27)
+				)
+				(hide yes)
 			)
 		)
@@
 			(at 106.68 92.71 0)
 			(effects
+				(font
+					(size 1.27 1.27)
+				)
+				(hide yes)
+			)
+		)
+		(property "Manufacturer" "TI"
+			(at 106.68 92.71 0)
+			(effects
+				(font
+					(size 1.27 1.27)
+				)
+				(hide yes)
+			)
+		)
+		(property "MPN" "TS5A3159DCK"
+			(at 106.68 92.71 0)
+			(effects
